File: MP3-Player/DAC.kicad_sch (KiCad schematic)
At the start: 1 part, among them J501 AudioJack3

Commit message: Added all schematic symbols. Time to start wiring up!
Parts:
- added U501: TAD5242, symbol MP3-Player_Symbol_Libraries:TAD5242
Other:
- moved on the sheet: J501
Changed lines of the file:
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@@
 	(symbol
 		(lib_id "Connector_Audio:AudioJack3")
-		(at 114.3 62.23 0)
+		(at 137.16 67.31 0)
 		(unit 1)
 		(exclude_from_sim no)
@@
 		(fields_autoplaced yes)
 		(property "Reference" "J501"
-			(at 112.395 53.34 0)
+			(at 135.255 58.42 0)
 			(effects
 				(font
@@
 		)
 		(property "Value" "AudioJack3"
-			(at 112.395 55.88 0)
+			(at 135.255 60.96 0)
 			(effects
 				(font
@@
 		)
 		(property "Footprint" ""
-			(at 114.3 62.23 0)
+			(at 137.16 67.31 0)
 			(effects
 				(font
@@
 		)
 		(property "Datasheet" "~"
-			(at 114.3 62.23 0)
+			(at 137.16 67.31 0)
 			(effects
 				(font
@@
 		)
 		(property "Description" "Audio Jack, 3 Poles (Stereo / TRS)"
-			(at 114.3 62.23 0)
+			(at 137.16 67.31 0)
 			(effects
 				(font
@@
 					(unit 1)
 				)
+			)
+		)
+	)
+	(symbol
+		(lib_id "MP3-Player_Symbol_Libraries:TAD5242")
+		(at 91.44 55.88 0)
+		(unit 1)
+		(exclude_from_sim no)
+		(in_bom yes)
+		(on_board yes)
+		(dnp no)
+		(fields_autoplaced yes)
+		(property "Reference" "U501"
+			(at 96.1233 50.8 0)
+			(effects
+				(font
+					(size 1.27 1.27)
+				)
+				(justify left)
+			)
+		)
+		(property "Value" "TAD5242"
+			(at 96.1233 53.34 0)
+			(effects
+				(font
+					(size 1.27 1.27)
+				)
+				(justify left)
+			)
+		)
+		(property "Footprint" ""
+			(at 91.44 55.88 0)
+			(effects
+				(font
+					(size 1.27 1.27)
+				)
+				(hide yes)
+			)
+		)
+		(property "Datasheet" ""
+			(at 91.44 55.88 0)
+			(effects
+				(font
+					(size 1.27 1.27)
+				)
+				(hide yes)
+			)
+		)
+		(property "Description" ""
+			(at 91.44 55.88 0)
+			(effects
+				(font
+					(size 1.27 1.27)
+				)
+				(hide yes)
+			)
+		)
+		(pin "16"
+		)
+		(pin "A2"
+		)
+		(pin "A4"
+		)
+		(pin "18"
+		)
+		(pin "21"
+		)
+		(pin "15"
+		)
+		(pin "13"
+		)
+		(pin "24"
+		)
+		(pin "12"
+		)
+		(pin "10"
+		)
+		(pin "9"
+		)
+		(pin "8"
+		)
+		(pin "7"
+		)
+		(pin "4"
+		)
+		(pin "1"
+		)
+		(pin "5"
+		)
+		(pin "23"
+		)
+		(pin "19"
+		)
+		(pin "2"
+		)
+		(pin "3"
+		)
+		(pin "14"
+		)
+		(pin "22"
+		)
+		(pin "A1"
+		)
+		(pin "A3"
+		)
+		(pin "11"
+		)
+		(pin "20"
+		)
+		(pin "6"
+		)
+		(pin "17"
+		)
+		(instances
+			(project ""
+				(path "/3f51ea9b-d2e1-4711-a47c-269e1b97e0f4/55939feb-9632-43ca-a0aa-b7cf8cf1876d"
+					(reference "U501")
+					(unit 1)
+				)
