File: MP3-Player/Peripherals.kicad_sch (KiCad schematic)
At the start: 3 parts

Commit message: Added all schematic symbols. Time to start wiring up!
Parts:
- added Q401: AO3401A, Package_TO_SOT_SMD:SOT-23, symbol Transistor_FET:AO3401A
- added SW401, SW402, SW403, SW404: 1-1825910-4, symbol Switch:SW_MEC_5E
- gave numbers to parts that had none: 3
