File: MP3-Player/Power.kicad_sch (KiCad schematic)
At the start: 2 parts, among them U302 TLV73333PDBV

Commit message: Added all schematic symbols. Time to start wiring up!
Parts:
- added J301: Conn_01x02_Socket, symbol Connector:Conn_01x02_Socket
- U301: value ~ -> BQ24259
Changed lines of the file:
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@@
 	(paper "A4")
+	(symbol
+		(lib_id "Connector:Conn_01x02_Socket")
+		(at 170.18 83.82 0)
+		(unit 1)
+		(exclude_from_sim no)
+		(in_bom yes)
+		(on_board yes)
+		(dnp no)
+		(fields_autoplaced yes)
+		(property "Reference" "J301"
+			(at 171.45 83.8199 0)
+			(effects
+				(font
+					(size 1.27 1.27)
+				)
+				(justify left)
+			)
+		)
+		(property "Value" "Conn_01x02_Socket"
+			(at 171.45 86.3599 0)
+			(effects
+				(font
+					(size 1.27 1.27)
+				)
+				(justify left)
+			)
+		)
+		(property "Footprint" ""
+			(at 170.18 83.82 0)
+			(effects
+				(font
+					(size 1.27 1.27)
+				)
+				(hide yes)
+			)
+		)
+		(property "Datasheet" "~"
+			(at 170.18 83.82 0)
+			(effects
+				(font
+					(size 1.27 1.27)
+				)
+				(hide yes)
+			)
+		)
+		(property "Description" "Generic connector, single row, 01x02, script generated"
+			(at 170.18 83.82 0)
+			(effects
+				(font
+					(size 1.27 1.27)
+				)
+				(hide yes)
+			)
+		)
+		(pin "2"
+		)
+		(pin "1"
+		)
+		(instances
+			(project ""
+				(path "/3f51ea9b-d2e1-4711-a47c-269e1b97e0f4/156723cf-95cb-4e74-b8dc-320a10f9d20f"
+					(reference "J301")
+					(unit 1)
+				)
+			)
+		)
+	)
 	(symbol
 		(lib_id "Regulator_Linear:TLV73333PDBV")
@@
 	(symbol
 		(lib_id "MP3-Player_Symbol_Libraries:BQ24259")
-		(at 80.01 46.99 0)
+		(at 81.28 48.26 0)
 		(unit 1)
 		(exclude_from_sim no)
@@
 		(fields_autoplaced yes)
 		(property "Reference" "U301"
-			(at 80.645 40.64 0)
-			(effects
-				(font
-					(size 1.27 1.27)
-				)
-			)
-		)
-		(property "Value" "~"
-			(at 80.645 43.18 0)
+			(at 81.915 40.64 0)
+			(effects
+				(font
+					(size 1.27 1.27)
+				)
+			)
+		)
+		(property "Value" "BQ24259"
+			(at 81.915 43.18 0)
 			(effects
 				(font
@@
 		)
 		(property "Footprint" ""
-			(at 80.01 46.99 0)
+			(at 81.28 48.26 0)
 			(effects
 				(font
@@
 		)
 		(property "Datasheet" ""
-			(at 80.01 46.99 0)
+			(at 81.28 48.26 0)
 			(effects
 				(font
@@
 		)
 		(property "Description" ""
-			(at 80.01 46.99 0)
-			(effects
-				(font
-					(size 1.27 1.27)
-				)
-				(hide yes)
-			)
+			(at 81.28 48.26 0)
+			(effects
+				(font
+					(size 1.27 1.27)
+				)
+				(hide yes)
+			)
+		)
+		(pin "18"
+		)
+		(pin "13"
+		)
+		(pin "16"
+		)
+		(pin "20"
+		)
+		(pin "17"
+		)
+		(pin "1"
+		)
+		(pin "19"
+		)
+		(pin "14"
+		)
+		(pin "10"
+		)
+		(pin "12"
+		)
+		(pin "21"
+		)
+		(pin "5"
+		)
+		(pin "9"
+		)
+		(pin "7"
+		)
+		(pin "15"
+		)
+		(pin "6"
+		)
+		(pin "22"
+		)
+		(pin "11"
+		)
+		(pin "4"
+		)
+		(pin "8"
+		)
+		(pin "23"
+		)
+		(pin "24"
+		)
+		(pin "3"
 		)
 		(pin "2"
 		)
-		(pin "5"
-		)
-		(pin "11"
-		)
-		(pin "1"
-		)
-		(pin "7"
-		)
-		(pin "22"
-		)
-		(pin "13"
-		)
-		(pin "6"
-		)
-		(pin "3"
-		)
-		(pin "4"
-		)
-		(pin "10"
-		)
-		(pin "15"
-		)
-		(pin "21"
-		)
-		(pin "19"
-		)
-		(pin "8"
-		)
-		(pin "20"
-		)
-		(pin "23"
-		)
-		(pin "24"
-		)
-		(pin "12"
-		)
-		(pin "17"
-		)
-		(pin "14"
-		)
-		(pin "16"
-		)
-		(pin "9"
-		)
-		(pin "18"
-		)
 		(instances
